File: pcbs/adaptador/ps2-nes/ps2-nes.kicad_sch (KiCad schematic)
At the start: 0 parts

Commit message: Fixing the 3d model screen dimensions.
Parts:
- added J1: PS2 Controller_pins, Package_SO:TI_SO-PowerPAD-8_ThermalVias, symbol Connector:DIN-6
- added J2: NES Contoller_pins, Connector:Tag-Connect_TC2030-IDC-NL_2x03_P1.27mm_Vertical, symbol Connector:Conn_01x07_Pin
- added R1: R, Resistor_THT:R_Array_SIP4, symbol Device:R_Small
Connections:
- new net: J2.1 (Pin_1), R1.1
- new net +5V: J1.4, J2.2 (Pin_2)
- new net Clock: J1.5, J2.3 (Pin_3)
- new net Data: J1.1, J2.4 (Pin_4)
- new net GND: J1.3, J2.5 (Pin_5), R1.2
- no-connect marks 0 -> 4
